File: kicad_files/keeb.kicad_pcb (KiCad board)
At the start: 2 copper layers, 3.6 x 3.2 mm, 230 parts, among them SW10 SW_Push, SW11 SW_Push, SW12 SW_Push, SW13 SW_Push, SW14 SW_Push, SW15 SW_Push, SW16 SW_Push, SW17 SW_Push, SW18 SW_Push, SW19 SW_Push, SW2 RotaryEncoder_Switch, SW20 SW_Push, SW21 SW_Push, SW22 SW_Push, SW23 SW_Push, SW24 SW_Push, SW25 SW_Push, SW26 SW_Push, SW27 SW_Push, SW28 SW_Push, SW29 SW_Push, SW3 SW_Push, SW30 SW_Push, SW31 SW_Push, SW32 SW_Push, SW33 SW_Push, SW34 SW_Push, SW35 SW_Push, SW36 SW_Push, SW37 SW_Push, SW38 SW_Push, SW39 SW_Push, SW4 SW_Push, SW40 SW_Push, SW41 SW_Push, SW42 SW_Push, SW43 SW_Push, SW44 SW_Push, SW45 SW_Push, SW46 SW_Push, SW47 SW_Push, SW48 SW_Push, SW49 SW_Push, SW5 SW_Push, SW50 SW_Push, SW51 SW_Push, SW52 SW_Push, SW53 SW_Push, SW54 SW_Push, SW55 SW_Push, SW56 SW_Push, SW6 SW_Push, SW7 SW_Push, SW8 SW_Push, SW9 SW_Push, U2 ER_OLEDM0.91_1x-I2C

Commit message: Started pcb
Parts:
- moved SW14 273.0 mm to (319.1, 38.4)
- moved SW26 260.9 mm to (319.1, 57.5)
- moved SW38 251.9 mm to (319.1, 76.5)
- moved C3 248.0 mm to (19.1, 41.3), turned to 90 degrees
- moved C9 246.4 mm to (19.1, 60.7), turned to 90 degrees
- moved C27 243.7 mm to (19.1, 117.9), turned to 90 degrees
- moved C15 243.5 mm to (19.1, 79.8), turned to 90 degrees
- moved C21 242.6 mm to (19.1, 98.8), turned to 90 degrees
- moved SW11 240.7 mm to (247.3, 38.4)
- moved SW13 238.9 mm to (285.4, 38.4)
- moved SW25 225.5 mm to (285.4, 57.5)
- moved D80 220.5 mm to (23.8, 119.1)
- moved SW12 220.2 mm to (266.4, 38.4)
- moved D62 219.3 mm to (23.8, 61.9)
- moved C4 218.5 mm to (52.4, 41.7), turned to 90 degrees
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
Commit message: PCB layout completed, routing needed
Parts:
- A1: moved to B.Cu
- S1, S2: footprint PCM_marbastlib-mx:STAB_MX_P_2u -> PCM_marbastlib-mx:STAB_MX_2u
- moved D106 324.1 mm to (350.6, 10.1), turned to 30 degrees
- moved D109 316.5 mm to (379.2, 59.6), turned to 30 degrees
- moved D108 310.8 mm to (369.7, 43.1), turned to 30 degrees
- moved D107 305.8 mm to (360.2, 26.6), turned to 30 degrees
- moved C58 291.3 mm to (374.5, 60.9), turned to 120 degrees
- moved D105 289.9 mm to (331.3, 43.3), turned to 30 degrees
- moved D112 288.2 mm to (350.3, 76.3), turned to 30 degrees
- moved C59 288.1 mm to (365.0, 44.4), turned to 120 degrees
- moved C60 286.4 mm to (355.4, 27.9), turned to 120 degrees
- moved D104 286.3 mm to (321.8, 26.8), turned to 30 degrees
- moved D99 286.1 mm to (331.5, 81.7), turned to 30 degrees
- moved C61 285.1 mm to (344.9, 12.0), turned to 120 degrees
- moved D111 282.9 mm to (340.8, 59.8), turned to 30 degrees
- moved D98 280.8 mm to (321.9, 65.2), turned to 30 degrees
- moved D89 268.4 mm to (314.9, 119.7), turned to 30 degrees
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Connections:
- SW51 pad 1: /COL_0 -> /COL_3
- SW52 pad 1: /COL_1 -> /COL_4
- SW53 pad 1: /COL_2 -> /COL_5
- SW54 pad 1: /COL_9 -> /COL_6
- SW55 pad 1: /COL_10 -> /COL_7
- SW56 pad 1: /COL_11 -> /COL_8
Routing:
- net /ROW_0: track 0.00 -> 143.8 mm
- net /ROW_1: track 0.00 -> 130.1 mm, vias 0 -> 10
- net /COL_5: track 0.00 -> 97.9 mm
- net /COL_4: track 0.00 -> 91.6 mm
- net /COL_3: track 0.00 -> 91.3 mm
- net /COL_0: track 0.00 -> 58.1 mm
- net /COL_1: track 0.00 -> 57.1 mm
- net /COL_2: track 0.00 -> 57.1 mm
- net Net-(D15-~-Pad2): track 0.00 -> 7.02 mm
- net Net-(D3-~-Pad2): track 0.00 -> 7.02 mm
Other:
- board size 3.6 x 3.2 mm -> 356.9 x 197.8 mm

Commit message: PCB layout fixed fr this time I hope...
Parts:
- C10, C11, C12, C13, C14, C15, C16, C17, C18, C19, C20, C21, C22, C23, C24, C25, C26, C27, C28, C29, C3, C32, C34, C35, C36, C37, C38, C39, C4, C40, C42, C43, C44, C45, C47, C48, C49, C5, C50, C51, C52, C53, C54, C55, C56, C57, C58, C59, C6, C60, C61, C7, C8, C9, D10, D100, D101, D102, D103, D104, D105, D106, D107, D108, D109, D11, D110, D111, D112, D12, D13, D14, D15, D16, D17, D18, D19, D2, D20, D21, D22, D23, D24, D25, D26, D27, D28, D29, D3, D30, D31, D32, D33, D34, D35, D36, D37, D38, D39, D4, D40, D41, D43, D44, D45, D46, D47, D48, D49, D5, D50, D51, D52, D53, D54, D55, D56, D57, D58, D59, D6, D60, D61, D62, D63, D64, D65, D66, D67, D68, D69, D7, D70, D71, D72, D73, D74, D75, D76, D77, D78, D79, D8, D80, D81, D82, D83, D84, D85, D86, D88, D89, D9, D90, D91, D93, D94, D95, D96, D98, D99: moved to B.Cu
- moved D50 47.7 mm to (391.2, 100.3), turned to 105 degrees
- moved D38 46.5 mm to (386.3, 81.9), turned to 105 degrees
- moved D26 45.8 mm to (381.4, 63.5), turned to 105 degrees
- moved D14 45.6 mm to (376.4, 45.1), turned to 105 degrees
- moved D109 45.4 mm to (382.1, 104.9), turned to -165 degrees
- moved C21 45.4 mm to (35.0, 103.1), turned to 75 degrees
- moved SW50 45.1 mm to (381.1, 100.6), turned to 15 degrees
- moved D59 44.3 mm to (39.3, 105.5), turned to 165 degrees
- moved C58 44.1 mm to (377.2, 105.0), turned to 105 degrees
- moved D108 44.1 mm to (377.2, 86.5), turned to -165 degrees
- moved C15 44.1 mm to (39.9, 84.7), turned to 75 degrees
- moved SW38 43.9 mm to (376.2, 82.2), turned to 15 degrees
- moved SW39 43.8 mm to (40.8, 100.9), turned to -15 degrees
- moved C9 43.3 mm to (44.9, 66.3), turned to 75 degrees
- moved D107 43.2 mm to (372.2, 68.1), turned to -165 degrees
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Routing:
- net /ROW_0: track 143.8 -> 0.00 mm
- net /ROW_1: track 130.1 -> 0.48 mm, vias 10 -> 0
- net /COL_5: track 97.9 -> 5.12 mm
- net /COL_4: track 91.6 -> 0.00 mm
- net /COL_3: track 91.3 -> 9.14 mm
- net /COL_1: track 57.1 -> 0.00 mm
- net /COL_2: track 57.1 -> 0.00 mm
- net /COL_0: track 58.1 -> 2.68 mm
- net Net-(D3-~-Pad2): track 7.02 -> 0.11 mm
- net Net-(D15-~-Pad2): track 7.02 -> 0.11 mm
Other:
- board size 356.9 x 197.8 mm -> 369.3 x 146.3 mm

Commit message: key matrix wiring
Parts:
- moved D64 5.13 mm to (103.9, 54.8)
- moved D30 5.13 mm to (123.4, 92.3)
- moved C44 5.13 mm to (276.8, 82.3)
- moved D91 5.13 mm to (258.1, 146.4)
- moved C29 5.13 mm to (163.6, 143.5)
- moved D37 5.13 mm to (351.9, 85.8)
- moved C53 5.13 mm to (308.6, 54.0)
- moved H5 5.13 mm to (70.1, 42.9)
- moved D84 5.13 mm to (264.5, 91.7)
- moved D85 5.13 mm to (269.4, 110.1)
- moved D82 5.13 mm to (159.4, 145.7)
- moved C38 5.13 mm to (279.9, 151.3)
- moved C12 5.13 mm to (114.3, 71.1)
- moved D50 5.13 mm to (389.3, 95.5)
- moved D8 5.13 mm to (167.7, 74.2)
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Routing:
- net /ROW_3: track 0.00 -> 414.0 mm, vias 0 -> 12
- net /ROW_2: track 0.00 -> 392.7 mm, vias 0 -> 22
- net /ROW_1: track 0.48 -> 369.4 mm, vias 0 -> 22
- net /ROW_0: track 0.00 -> 358.3 mm, vias 0 -> 23
- net /COL_11: track 0.00 -> 319.2 mm, vias 0 -> 2
- net /ROW_4: track 0.00 -> 266.4 mm
- net /COL_10: track 0.00 -> 254.5 mm, vias 0 -> 2
- net /COL_4: track 0.00 -> 251.0 mm
- net /COL_0: track 2.68 -> 239.6 mm
- net /COL_1: track 0.00 -> 201.8 mm
- net /COL_3: track 9.14 -> 199.4 mm
- net /COL_2: track 0.00 -> 185.1 mm
- net /COL_8: track 0.00 -> 177.0 mm
- net /COL_5: track 5.12 -> 168.2 mm
- net /COL_9: track 0.00 -> 162.5 mm, vias 0 -> 2
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Other:
- board size 369.3 x 146.3 mm -> 369.3 x 148.8 mm

Commit message: RGB kinda done, need to find a way to do the ground well
Parts:
- moved D77 99.1 mm to (131.9, 169.4)
- moved D60 75.4 mm to (69.0, 127.9)
- moved D68 75.4 mm to (108.2, 128.9)
- moved D78 72.4 mm to (158.9, 164.4), turned to 45 degrees
- moved D63 49.4 mm to (103.4, 73.4)
- moved D72 37.4 mm to (135.3, 101.3)
- moved D61 37.4 mm to (74.0, 109.5)
- moved D69 37.4 mm to (113.2, 110.5)
- moved D74 28.5 mm to (123.0, 73.7)
- moved D65 27.0 mm to (78.9, 91.1)
- moved D64 27.0 mm to (83.8, 72.7)
- moved D81 26.4 mm to (147.6, 129.3)
- moved D62 24.0 mm to (98.5, 91.8)
- moved D71 23.6 mm to (130.4, 119.7)
- moved D79 20.4 mm to (157.4, 92.4)
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Routing:
- net +5V: track 0.00 -> 1815.8 mm, vias 0 -> 58
- net /LED_MATRIX_LEFT/DOUT: track 0.00 -> 350.2 mm, vias 0 -> 2
- net /LED_DATA: track 0.00 -> 78.3 mm, vias 0 -> 3
- net Net-(D103-DOUT): track 0.00 -> 50.1 mm
- net Net-(D59-DOUT): track 0.00 -> 46.1 mm
- net Net-(D109-DIN): track 0.00 -> 46.1 mm
- net Net-(D63-DIN): track 0.00 -> 42.8 mm, vias 0 -> 2
- net Net-(D76-DOUT): track 0.00 -> 41.4 mm
- net Net-(D67-DOUT): track 0.00 -> 40.5 mm, vias 0 -> 2
- net Net-(D100-DOUT): track 0.00 -> 40.2 mm
- net Net-(D95-DOUT): track 0.00 -> 39.5 mm
- net Net-(D89-DIN): track 0.00 -> 39.1 mm
- net Net-(D80-DIN): track 0.00 -> 38.7 mm, vias 0 -> 4
- net Net-(D70-DOUT): track 0.00 -> 37.3 mm, vias 0 -> 2
- net Net-(D68-DOUT): track 0.00 -> 36.7 mm
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
Commit message: pcb done yay yay yippee
Parts:
- added G***: LOGO, LOGO, F.Cu at (47.7, 87.3)
- moved SW15 8.86 mm to (47.2, 69.2)
- moved D19 8.86 mm to (144.0, 92.9)
- moved D50 8.86 mm to (387.7, 105.3)
- moved D110 8.86 mm to (297.3, 82.5)
- moved D8 8.86 mm to (166.1, 84.0)
- moved H7 8.86 mm to (346.0, 52.1)
- moved SW6 8.86 mm to (123.2, 60.3)
- moved D67 8.86 mm to (87.5, 119.8)
- moved C7 8.86 mm to (134.9, 71.7)
- moved D100 8.86 mm to (307.1, 119.3)
- moved C37 8.86 mm to (260.6, 159.4)
- moved D61 8.86 mm to (72.9, 100.7)
- moved SW17 8.86 mm to (98.6, 78.4)
- moved SW37 8.86 mm to (340.2, 95.9)
- moved SW40 8.86 mm to (69.2, 114.5)
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Routing:
- net GND: track 0.00 -> 669.2 mm, vias 0 -> 149
- net (no net): track 0.00 -> 2.38 mm, vias 0 -> 2
- net /SCL: track 26.7 -> 27.8 mm
- net /VCC: track 55.6 -> 56.6 mm
- net /COL_11: track 319.2 -> 319.7 mm
- added copper zone on B.Cu, net GND
Other:
- board text added: "Lmaoo"

Commit message: Added gerbers, bom
Routing:
- net /COL_2: track 189.1 -> 180.7 mm
- net /LED_MATRIX_LEFT/DOUT: track 350.2 -> 346.4 mm, vias 2 -> 4
- net +5V: track 1815.7 -> 1813.4 mm
- net GND: track 669.2 -> 670.3 mm
Other:
- outline, holes or cut-outs redrawn
